File: hw/roamr-power/12v_to_3v3.kicad_sch (KiCad schematic)
At the start: 0 parts

Commit message: reorganizing to roamr-power
Other:
- title: (none) -> ROAMR power board
Changed lines of the file:
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@@
 	(generator_version "9.0")
 	(paper "USLetter")
+	(title_block
+		(title "ROAMR power board")
+		(date "2026-01-18")
+		(rev "1.0")
+	)
 	(text "12V to 3V3 buck here"
 		(exclude_from_sim no)
