File: hw/roamr-power/connectors.kicad_sch (KiCad schematic)
At the start: 0 parts

Commit message: reorganizing to roamr-power
Other:
- title: (none) -> ROAMR power board
Changed lines of the file:
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@@
 	(generator_version "9.0")
 	(paper "USLetter")
+	(title_block
+		(title "ROAMR power board")
+		(date "2026-01-18")
+		(rev "1.0")
+	)
 	(text "so in total we need 5 connectors:\n- battery in\n- 12V out\n- 5V out\n- 3V3 out\n- USB out"
 		(exclude_from_sim no)
