File: hw/roamr-power/roamr-power.kicad_pcb (KiCad board)
At the start: 0 parts

Commit message: picked the BOM and added two more indicator LEDs for the 12V and 5V rails
Parts:
- added C1: 0.1uF, Capacitor_SMD:C_0603_1608Metric, F.Cu at (149.3, 56.1)
- added C10: 22.0uF, Capacitor_SMD:C_0603_1608Metric, F.Cu at (153.3, 61.1)
- added C11: 39.0uF, 35SVPF39M:16SVF270M, F.Cu at (140.2, 72.0)
- added C12: 120uF, GYG1E121MCQ1GS:CAPAE660X610N, F.Cu at (142.6, 89.3)
- added C13: 0.1uF, Capacitor_SMD:C_0603_1608Metric, F.Cu at (135.1, 86.2)
- added C14: 0.1uF, Capacitor_SMD:C_0603_1608Metric, F.Cu at (135.1, 88.7)
- added C3: 150.0pF, Capacitor_SMD:C_0603_1608Metric, F.Cu at (149.3, 58.6)
- added C4: 22.0uF, Capacitor_SMD:C_0603_1608Metric, F.Cu at (149.3, 61.1)
- added C5: 1.0uF, Capacitor_SMD:C_0603_1608Metric, F.Cu at (149.3, 63.7)
- added C6: 15.0uF, Capacitor_SMD:C_0603_1608Metric, F.Cu at (149.3, 66.2)
- added C7: 4.7uF, Capacitor_SMD:C_0603_1608Metric, F.Cu at (153.3, 56.1)
- added C8: 39.0uF, 35SVPF39M:16SVF270M, F.Cu at (140.2, 60.6)
- added C9: 4.7uF, Capacitor_SMD:C_0603_1608Metric, F.Cu at (153.3, 58.6)
- added D1: 1N5819, Diode_THT:D_DO-41_SOD81_P10.16mm_Horizontal, F.Cu at (101.9, 70.5)
- added D2: GLED, KT_EELP41.12-S2U1-25-2X4X-5-R18:KTEELP4112S2U1252X4X5R18, F.Cu at (149.8, 102.0)
- added D3: RLED, KR_DELPS1.22-VGVI-23-H3Q4:KRDELPS122VGVI23H3Q4, F.Cu at (144.5, 102.0)
- added D4: 1N5819, Diode_THT:D_DO-41_SOD81_P10.16mm_Horizontal, F.Cu at (101.9, 74.8)
- added D5: 1N5819, Diode_THT:D_DO-41_SOD81_P10.16mm_Horizontal, F.Cu at (101.9, 79.0)
- added D6: D_TVS, SMLJ12A-R:DIOM7959X262N, F.Cu at (119.3, 83.0)
- added D7: GLED, KT_EELP41.12-S2U1-25-2X4X-5-R18:KTEELP4112S2U1252X4X5R18, F.Cu at (158.4, 77.1)
- added D8: GLED, KT_EELP41.12-S2U1-25-2X4X-5-R18:KTEELP4112S2U1252X4X5R18, F.Cu at (158.4, 81.0)
- added J1: Conn_01x02_Socket, TB002-500-02BE:TB00250002BE, F.Cu at (118.2, 74.1)
- added J2: Conn_01x02_Socket, Connector_JST:JST_XH_S2B-XH-A-1_1x02_P2.50mm_Horizontal, F.Cu at (103.5, 59.8)
- added J3: Conn_01x02_Socket, Connector_JST:JST_XH_S2B-XH-A-1_1x02_P2.50mm_Horizontal, F.Cu at (113.0, 59.8)
- added L1: 3.3uH, ETQ-P4M3R3YFN:IND_PCC-M0645M_PAN-L, F.Cu at (151.5, 79.0)
- added L2: 4.7uH, VLS6045EX_4R7M:IND_VLS6045EX-4R7M_TDK-L, F.Cu at (152.2, 71.3)
- added P2: USB_C_Plug_USB2.0, USB4125-GF-A:CONN6_USB4125_GCT, F.Cu at (125.3, 60.9)
- added Q1: Q_PMOS_DSG, BSS84PH6327XTSA2:SOT95P240X110-3N, F.Cu at (139.5, 102.3)
- added R1: 52.3kR, Resistor_SMD:R_0603_1608Metric, F.Cu at (153.3, 63.7)
- added R10: 510R, Resistor_SMD:R_0603_1608Metric, F.Cu at (157.3, 63.7)
- added R2: 24kR, Resistor_SMD:R_0603_1608Metric, F.Cu at (135.1, 91.2)
- added R3: 73.2kR, Resistor_SMD:R_0603_1608Metric, F.Cu at (153.3, 66.2)
- added R4: 10.0kR, Resistor_SMD:R_0603_1608Metric, F.Cu at (157.3, 56.1)
- added R5: 1.8kR, Resistor_SMD:R_0603_1608Metric, F.Cu at (157.3, 58.6)
- added R6: 1.3R, Resistor_SMD:R_0603_1608Metric, F.Cu at (157.3, 61.1)
- added R7: 510R, Resistor_SMD:R_0603_1608Metric, F.Cu at (135.1, 93.7)
- added R8: 560R, Resistor_SMD:R_0603_1608Metric, F.Cu at (135.1, 96.2)
- added R9: 100kR, Resistor_SMD:R_0603_1608Metric, F.Cu at (135.1, 98.7)
- added SW1: SW_SPDT, OS102011MS2QN1:OS102011MA1QN1, F.Cu at (142.8, 97.3)
- added TP1: TestPoint, TestPoint:TestPoint_Pad_D1.5mm, F.Cu at (129.3, 70.2)
- added TP2: TestPoint, TestPoint:TestPoint_Pad_D1.5mm, F.Cu at (129.3, 73.7)
- added TP3: TestPoint, TestPoint:TestPoint_Keystone_5005-5009_Compact, F.Cu at (102.6, 83.7)
- added TP4: TestPoint, TestPoint:TestPoint_Pad_D1.5mm, F.Cu at (129.3, 77.3)
- added U1: TPS56A37RPAR, TPS56A37RPAR:RPA0010A-MFG, F.Cu at (136.1, 79.9)
- added U2: TPS2553DDBVR, TPS2553DDBVR:DRV6_1P6X1_TEX, F.Cu at (150.3, 86.8)
Other:
- board outline added: 8.7 x 4.4 mm
- copper layers 0 -> 2
