File: hw/roamr-power/roamr-power.kicad_pcb (KiCad board)
At the start: 2 copper layers, 8.7 x 4.4 mm, 45 parts, among them J1 Conn_01x02_Socket, J2 Conn_01x02_Socket, J3 Conn_01x02_Socket, P2 USB_C_Plug_USB2.0, Q1 Q_PMOS_DSG, SW1 SW_SPDT, U1 TPS56A37RPAR, U2 TPS2553DDBVR

Commit message: layout
Parts:
- added NT1: NetTie_2, NetTie:NetTie-2_SMD_Pad0.5mm, F.Cu at (134.7, 71.0)
- L2: footprint VLS6045EX_4R7M:IND_VLS6045EX-4R7M_TDK-L -> VLS6045EX_4R7M:IND_VLS6045EX-4R7M_TDK
- P2: footprint USB4125-GF-A:CONN6_USB4125_GCT -> USB4125-GF-A:USB4125GFA
- U2: footprint TPS2553DDBVR:DRV6_1P6X1_TEX -> TPS2553DDBVR:SOT95P280X145-6N
- moved J2 72.7 mm to (176.2, 63.8), turned to 90 degrees
- moved J3 66.3 mm to (176.2, 79.8), turned to 90 degrees
- moved D4 66.0 mm to (167.5, 67.7), turned to 90 degrees
- moved D5 65.7 mm to (167.5, 83.6), turned to 90 degrees
- moved C12 55.7 mm to (88.8, 75.2), turned to 90 degrees
- moved P2 55.6 mm to (72.6, 78.5), turned to -90 degrees
- moved SW1 53.4 mm to (90.5, 86.5), turned to 180 degrees
- moved U2 51.3 mm to (100.2, 76.0)
- moved D2 48.1 mm to (104.0, 87.0), turned to 90 degrees
- moved J1 47.6 mm to (72.5, 60.9), turned to -90 degrees
- moved D3 46.0 mm to (101.0, 87.1), turned to 90 degrees
- moved Q1 44.9 mm to (100.3, 80.5), turned to 180 degrees
- moved R9 42.6 mm to (96.2, 81.5)
- moved R2 41.3 mm to (96.2, 77.5), turned to 180 degrees
- moved D6 41.0 mm to (82.5, 65.0), turned to 90 degrees
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Connections:
- net Net-(D1-K) renamed /USB_OUT
- net Net-(D4-K) renamed /12V_OUT
- net Net-(D5-K) renamed /5V_OUT
- net Net-(U1-SW) renamed /12V to 5V/SW_OUT
- net Net-(U1-VIN) renamed /12V to 5V/12V_SW
- C10 pad 1: Net-(C10-Pad1) -> +5V
- C11 pad 1: Net-(C11-Pad1) -> +12V
- C4 pad 2: Net-(C10-Pad1) -> GND
- C7 pad 2: Net-(C7-Pad2) -> GND
- C8 pad 2: Net-(C11-Pad1) -> GND
- C9 pad 1: Net-(C7-Pad2) -> Net-(C7-Pad1)
Routing:
- net /Phone Charging/CHG_EN: track 0.00 -> 22.8 mm
- net +5V: track 0.00 -> 16.3 mm, vias 0 -> 2
- net VCTRL_5V: track 0.00 -> 15.1 mm
- net /12V_OUT: track 0.00 -> 10.3 mm
- net /5V_OUT: track 0.00 -> 10.2 mm
- net Net-(Q1-S): track 0.00 -> 6.23 mm, vias 0 -> 2
- net /Phone Charging/CURR_LIM_nFLT: track 0.00 -> 5.21 mm
- net GND: track 0.00 -> 4.70 mm, vias 0 -> 5
- net Net-(D8-A): track 0.00 -> 3.22 mm
- net Net-(D7-A): track 0.00 -> 3.08 mm
- net Net-(D2-A): track 0.00 -> 3.02 mm
- net Net-(D3-A): track 0.00 -> 2.86 mm
- net Net-(U2-ILIM): track 0.00 -> 2.64 mm
- net Net-(U1-BOOT): track 0.00 -> 2.46 mm
- net Net-(U1-FB): track 0.00 -> 1.90 mm
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- added copper zone on F.Cu, net +12V
- added copper zone on F.Cu, net +5V
- added copper zone on F.Cu, net /12V to 5V/12V_SW
- added copper zone on F.Cu, net /12V to 5V/SW_OUT
- added copper zone on F.Cu, net /USB_OUT
- added copper zone on B.Cu, net GND
- added copper zone on F.Cu, net GND
- added copper zone on F.Cu, net GNDA
- added copper zone on F.Cu, net VCTRL_5V
Other:
- board size 8.7 x 4.4 mm -> 115 x 55 mm

Commit message: pcb schematic and layout updated
Parts:
- added R11: 510R, Resistor_SMD:R_0603_1608Metric, F.Cu at (94.5, 61.5)
- added R12: 10kR, Resistor_SMD:R_0603_1608Metric, F.Cu at (96.3, 61.5)
- added R13: 10kR, Resistor_SMD:R_0603_1608Metric, F.Cu at (88.7, 61.5)
- added R14: 7.5kR, Resistor_SMD:R_0603_1608Metric, F.Cu at (87.0, 61.5)
- added R15: 56kR, Resistor_SMD:R_0603_1608Metric, F.Cu at (78.3, 77.8)
- added SW2: SW_SPDT, OS102011MS2QN1:OS102011MA1QN1, F.Cu at (90.7, 54.2)
- added U3: TPS259541DSGR, TPS259541DSGR:SON50P200X200X80-9N, F.Cu at (91.6, 62.9)
- D1, D4, D5: value 1N5819 -> PMEG3050EP,115; footprint Diode_THT:D_DO-41_SOD81_P10.16mm_Horizontal -> PMEG3050EP:PMEG3050EP115
- moved TP3 44.9 mm to (132.4, 80.4)
- moved D4 5.76 mm to (167.5, 61.9)
- moved D5 5.08 mm to (167.5, 78.5)
- moved D2 3.10 mm to (107.1, 86.8)
- moved D3 3.10 mm to (104.1, 87.0)
- moved R7 3.10 mm to (109.6, 86.5)
- moved R8 3.10 mm to (101.6, 86.5)
- moved D1 2.88 mm to (81.6, 76.3), turned to 90 degrees
- moved C12 2.51 mm to (89.8, 72.8)
- moved D6 2.19 mm to (81.6, 67.0)
- moved C13 1.57 mm to (103.2, 74.4)
- moved C14 1.45 mm to (96.2, 78.0)
- moved Q1 1.45 mm to (100.3, 79.0)
- moved R2 1.45 mm to (96.2, 76.0)
- moved R9 1.45 mm to (96.2, 80.0)
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Connections:
- net +5V renamed VSYS_5V
- net VCTRL_5V renamed VLIM_5V
- C11 pad 1: +12V -> VSYS_12V
- C8 pad 1: +12V -> VSYS_12V
- D4 pad 2: +12V -> VSYS_12V
- D6 pad 2: +12V -> VIN_12V
- J1 pad 1: +12V -> VIN_12V
- L2 pad 1: +12V -> VSYS_12V
- P2 pad A5: unconnected-(P2-CC-PadA5) -> Net-(P2-CC)
- R5 pad 1: +12V -> VSYS_12V
- TP1 pad 1: +12V -> VSYS_12V
Routing:
- net VIN_12V: track 0.00 -> 13.3 mm
- net /12V_OUT: track 10.3 -> 0.00 mm
- net /5V_OUT: track 10.2 -> 0.00 mm
- net /Phone Charging/CHG_EN: track 22.8 -> 29.3 mm
- net Net-(SW2-C): track 0.00 -> 6.45 mm
- net Net-(U3-~{FLT}): track 0.00 -> 3.88 mm
- net /VSYS_EN: track 0.00 -> 3.71 mm
- net Net-(P2-CC): track 0.00 -> 3.19 mm
- net Net-(Q1-S): track 6.23 -> 9.08 mm
- net Net-(U3-ILM): track 0.00 -> 1.88 mm
- net VLIM_5V: track 15.1 -> 14.5 mm
- net (no net): vias 1 -> 0
- added copper zone on F.Cu, net /12V_OUT
- added copper zone on F.Cu, net /5V_OUT
- added copper zone on F.Cu, net VIN_12V
- added copper zone on F.Cu, net VSYS_12V
- removed copper zone on F.Cu, net +12V
Other:
- board text added: "12V"
- board text added: "12V IN"
- board text added: "12V OUT"
- board text added: "5V"
- board text added: "5V 1A OUT"
- board text added: "5V OUT"
- board text added: "EN"
- board text added: "FLT"
- board text added: "GND"
- board text added: "OFF"
- board text added: "ON"
- board text added: "SYSTEM"
- board text added: "USB OUT"

Commit message: final changes
Parts:
- moved C3 0.70 mm to (133.1, 68.8)
- moved R3 0.70 mm to (130.7, 68.0)
- moved NT1 0.70 mm to (134.0, 71.0)
- moved R4 0.70 mm to (134.8, 68.8)
- moved R1 0.58 mm to (134.1, 66.5)
- moved L1 0.33 mm to (141.0, 73.9)
- moved C1 0.28 mm to (142.5, 68.5)
- moved C5 0.20 mm to (141.5, 63.8)
- moved C6 0.20 mm to (139.8, 63.8)
- moved C7 0.20 mm to (138.0, 60.5)
- moved C9 0.20 mm to (139.8, 60.6)
- moved R6 0.20 mm to (138.0, 63.7)
Routing:
- net VSYS_5V: track 16.3 -> 27.5 mm
- net Net-(U1-FB): track 1.90 -> 5.90 mm
- net Net-(U1-MODE): track 0.00 -> 2.80 mm
Changed lines of the file:
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@@
 	(footprint "Resistor_SMD:R_0603_1608Metric"
 		(layer "F.Cu")
-		(at 138 63.925 90)
+		(at 138 63.725 90)
 		(descr "Resistor SMD 0603 (1608 Metric), square (rectangular) end terminal, IPC-7351 nominal, (Body size source: IPC-SM-782 page 72, https://www.pcb-3d.com/wordpress/wp-content/uploads/ipc-sm-782a_amendment_1_and_2.pdf), generated with kicad-footprint-generator")
 		(tags "resistor")
@@
 	(footprint "Capacitor_SMD:C_0603_1608Metric"
 		(layer "F.Cu")
-		(at 139.75 60.775 90)
+		(at 139.75 60.575 90)
 		(descr "Capacitor SMD 0603 (1608 Metric), square (rectangular) end terminal, IPC-7351 nominal, (Body size source: IPC-SM-782 page 76, https://www.pcb-3d.com/wordpress/wp-content/uploads/ipc-sm-782a_amendment_1_and_2.pdf), generated with kicad-footprint-generator")
 		(tags "capacitor")
@@
 	(footprint "Capacitor_SMD:C_0603_1608Metric"
 		(layer "F.Cu")
-		(at 142.225 68.5)
+		(at 142.5 68.5)
 		(descr "Capacitor SMD 0603 (1608 Metric), square (rectangular) end terminal, IPC-7351 nominal, (Body size source: IPC-SM-782 page 76, https://www.pcb-3d.com/wordpress/wp-content/uploads/ipc-sm-782a_amendment_1_and_2.pdf), generated with kicad-footprint-generator")
 		(tags "capacitor")
@@
 	(footprint "ETQ-P4M3R3YFN:IND_PCC-M0645M_PAN-L"
 		(layer "F.Cu")
-		(at 141 73.6138 -90)
+		(at 141 73.9416 -90)
 		(tags "ETQP4M3R3YFN ")
 		(property "Reference" "L1"
@@
 			(layer "F.Paste")
 		)
+		(fp_rect
+			(start -2.75 -2.25)
+			(end 2.3 2.2)
+			(stroke
+				(width 0.05)
+				(type default)
+			)
+			(fill no)
+			(layer "F.CrtYd")
+		)
 		(fp_line
 			(start -1.549999 -1.549999)
@@
 	(footprint "Capacitor_SMD:C_0603_1608Metric"
 		(layer "F.Cu")
-		(at 141.5 63.975 90)
+		(at 141.5 63.775 90)
 		(descr "Capacitor SMD 0603 (1608 Metric), square (rectangular) end terminal, IPC-7351 nominal, (Body size source: IPC-SM-782 page 76, https://www.pcb-3d.com/wordpress/wp-content/uploads/ipc-sm-782a_amendment_1_and_2.pdf), generated with kicad-footprint-generator")
 		(tags "capacitor")
@@
 	(footprint "Resistor_SMD:R_0603_1608Metric"
 		(layer "F.Cu")
-		(at 135.5 68.825 90)
+		(at 134.8 68.825 90)
 		(descr "Resistor SMD 0603 (1608 Metric), square (rectangular) end terminal, IPC-7351 nominal, (Body size source: IPC-SM-782 page 72, https://www.pcb-3d.com/wordpress/wp-content/uploads/ipc-sm-782a_amendment_1_and_2.pdf), generated with kicad-footprint-generator")
 		(tags "resistor")
@@
 	(footprint "NetTie:NetTie-2_SMD_Pad0.5mm"
 		(layer "F.Cu")
-		(at 134.7 71 -90)
+		(at 134 71 -90)
 		(descr "Net tie, 2 pin, 0.5mm square SMD pads")
 		(tags "net tie")
@@
 	(footprint "Capacitor_SMD:C_0603_1608Metric"
 		(layer "F.Cu")
-		(at 133.800483 68.836497 90)
+		(at 133.100483 68.836497 90)
 		(descr "Capacitor SMD 0603 (1608 Metric), square (rectangular) end terminal, IPC-7351 nominal, (Body size source: IPC-SM-782 page 76, https://www.pcb-3d.com/wordpress/wp-content/uploads/ipc-sm-782a_amendment_1_and_2.pdf), generated with kicad-footprint-generator")
 		(tags "capacitor")
@@
 	(footprint "Capacitor_SMD:C_0603_1608Metric"
 		(layer "F.Cu")
-		(at 139.75 63.9804 90)
+		(at 139.75 63.7804 90)
 		(descr "Capacitor SMD 0603 (1608 Metric), square (rectangular) end terminal, IPC-7351 nominal, (Body size source: IPC-SM-782 page 76, https://www.pcb-3d.com/wordpress/wp-content/uploads/ipc-sm-782a_amendment_1_and_2.pdf), generated with kicad-footprint-generator")
 		(tags "capacitor")
@@
 	(footprint "Capacitor_SMD:C_0603_1608Metric"
 		(layer "F.Cu")
-		(at 138 60.725 90)
+		(at 138 60.525 90)
 		(descr "Capacitor SMD 0603 (1608 Metric), square (rectangular) end terminal, IPC-7351 nominal, (Body size source: IPC-SM-782 page 76, https://www.pcb-3d.com/wordpress/wp-content/uploads/ipc-sm-782a_amendment_1_and_2.pdf), generated with kicad-footprint-generator")
 		(tags "capacitor")
@@
 	(footprint "Resistor_SMD:R_0603_1608Metric"
 		(layer "F.Cu")
-		(at 134.675 66.5)
+		(at 134.1 66.5)
 		(descr "Resistor SMD 0603 (1608 Metric), square (rectangular) end terminal, IPC-7351 nominal, (Body size source: IPC-SM-782 page 72, https://www.pcb-3d.com/wordpress/wp-content/uploads/ipc-sm-782a_amendment_1_and_2.pdf), generated with kicad-footprint-generator")
 		(tags "resistor")
@@
 	(footprint "Resistor_SMD:R_0603_1608Metric"
 		(layer "F.Cu")
-		(at 131.425 68 180)
+		(at 130.725 68 180)
 		(descr "Resistor SMD 0603 (1608 Metric), square (rectangular) end terminal, IPC-7351 nominal, (Body size source: IPC-SM-782 page 72, https://www.pcb-3d.com/wordpress/wp-content/uploads/ipc-sm-782a_amendment_1_and_2.pdf), generated with kicad-footprint-generator")
 		(tags "resistor")
@@
 	)
 	(gr_line
-		(start 133.800483 68)
-		(end 132.2 68)
-		(stroke
-			(width 0.2)
-			(type default)
-		)
-		(layer "F.Cu")
-		(net 2)
-	)
-	(gr_line
 		(start 101.55 75.5)
 		(end 99.05 75.5)
@@
 	)
 	(gr_line
-		(start 137.3 65.8)
-		(end 136 65.8)
-		(stroke
-			(width 0.2)
-			(type default)
-		)
-		(layer "F.Cu")
-		(net 16)
-	)
-	(gr_line
-		(start 135.6 68)
-		(end 133.8 68)
-		(stroke
-			(width 0.2)
-			(type default)
-		)
-		(layer "F.Cu")
-		(net 2)
-	)
-	(gr_line
-		(start 130.6 68)
-		(end 130.6 75.2)
-		(stroke
-			(width 0.4)
-			(type solid)
-		)
-		(layer "F.Cu")
-		(net 13)
-	)
-	(gr_line
-		(start 133.8 69.6)
-		(end 133.8 75.2)
-		(stroke
-			(width 0.4)
-			(type solid)
-		)
-		(layer "F.Cu")
-		(net 13)
-	)
-	(gr_line
-		(start 136 65.8)
-		(end 135.5 66.3)
-		(stroke
-			(width 0.2)
-			(type default)
-		)
-		(layer "F.Cu")
-		(net 16)
-	)
-	(gr_line
 		(start 138 63.1)
 		(end 138 61.5)
@@
 		(net 5)
 	)
-	(gr_line
-		(start 137.6 66.1)
-		(end 137.3 65.8)
-		(stroke
-			(width 0.2)
-			(type default)
-		)
-		(layer "F.Cu")
-		(net 16)
-	)
 	(gr_arc
 		(start 184 92.9)
@@
 	)
 	(segment
-		(start 135.6 68)
-		(end 136.294599 67.305401)
+		(start 133.100483 68.061497)
+		(end 134.738503 68.061497)
 		(width 0.2)
 		(layer "F.Cu")
@@
 	)
 	(segment
-		(start 136.294599 67.305401)
+		(start 135.494599 67.305401)
 		(end 137.110002 67.305401)
 		(width 0.2)
@@
 	)
 	(segment
-		(start 135.5 68)
-		(end 135.6 68)
+		(start 133.100483 68.061497)
+		(end 131.611497 68.061497)
+		(width 0.2)
+		(layer "F.Cu")
+		(net 2)
+	)
+	(segment
+		(start 134.738503 68.061497)
+		(end 134.8 68)
+		(width 0.2)
+		(layer "F.Cu")
+		(net 2)
+	)
+	(segment
+		(start 134.8 68)
+		(end 135.494599 67.305401)
+		(width 0.2)
+		(layer "F.Cu")
+		(net 2)
+	)
+	(segment
+		(start 131.611497 68.061497)
+		(end 131.55 68)
 		(width 0.2)
 		(layer "F.Cu")
@@
 	)
 	(segment
+		(start 129.9 68.1)
+		(end 129.9 68)
+		(width 0.2)
+		(layer "F.Cu")
+		(net 13)
+	)
+	(segment
 		(start 90.5 86.5)
 		(end 90.5 86.3)
@@
 	)
 	(segment
+		(start 133.100483 69.611497)
+		(end 131.411497 69.611497)
+		(width 0.2)
+		(layer "F.Cu")
+		(net 13)
+	)
+	(segment
+		(start 131.411497 69.611497)
+		(end 129.9 68.1)
+		(width 0.2)
+		(layer "F.Cu")
+		(net 13)
+	)
+	(segment
 		(start 90.5 86.3)
 		(end 91.4 85.4)
@@
 		(net 13)
 	)
+	(segment
+		(start 129.9 68)
+		(end 129.9 75.3)
+		(width 0.2)
+		(layer "F.Cu")
+		(net 13)
+	)
 	(via
 		(at 102.8 77.1)
@@
 	)
 	(segment
+		(start 135.269599 66.155401)
+		(end 134.925 66.5)
+		(width 0.2)
+		(layer "F.Cu")
+		(net 16)
+	)
+	(segment
+		(start 137.580001 66.155401)
+		(end 135.269599 66.155401)
+		(width 0.2)
+		(layer "F.Cu")
+		(net 16)
+	)
+	(segment
 		(start 99 74.5)
 		(end 98.55 74.5)
@@
 		(polygon
 			(pts
-				(xy 142.225 68) (xy 142.525 67.7) (xy 143.4 67.7) (xy 143.7 68) (xy 143.7 69.2) (xy 143 69.9) (xy 143 71.9)
-				(xy 142.7 72.2) (xy 139.2 72.2) (xy 139 72) (xy 139 70.5) (xy 138 69.5) (xy 138 68.3554) (xy 138.510002 67.845398)
+				(xy 142.425 68.2) (xy 142.925 67.7) (xy 143.6 67.7) (xy 143.9 68) (xy 143.9 69.1) (xy 143 70) (xy 143 72.2)
+				(xy 142.6 72.6) (xy 139.5 72.6) (xy 139 72.1) (xy 139 70.5) (xy 138 69.5) (xy 138 68.3554) (xy 138.510002 67.845398)
 				(xy 138.510002 67.555401) (xy 138.765403 67.3) (xy 139 67.3) (xy 139.2 67.5) (xy 139.2 69.25) (xy 139.35 69.4)
-				(xy 141.8 69.4) (xy 142.225 68.975)
+				(xy 141.8 69.4) (xy 142.425 68.775)
 			)
 		)

Commit message: final edits
Parts:
- removed P2: USB_C_Plug_USB2.0, USB4125-GF-A:USB4125GFA
- added G***: LOGO, LOGO, F.Cu at (156.8, 70.1)
- added J4: USB4125-GF-A, USB4125-GF-A:USB4125GFA, F.Cu at (72.7, 78.5)
- added R16: 56kR, Resistor_SMD:R_0603_1608Metric, F.Cu at (78.3, 80.1)
- C6: footprint Capacitor_SMD:C_0603_1608Metric -> Capacitor_SMD:C_0805_2012Metric
- D2, D7, D8: footprint KT_EELP41.12-S2U1-25-2X4X-5-R18:KTEELP4112S2U1252X4X5R18 -> KT-0603:LEDC1608X70N
- D3: footprint KR_DELPS1.22-VGVI-23-H3Q4:KRDELPS122VGVI23H3Q4 -> KT-0603:LEDC1608X70N
- D6: value D_TVS -> SMLJ13A; footprint SMLJ12A-R:DIOM7959X262N -> SMLJ13CA-R:DIOM7959X262N
- J1: value Conn_01x02_Socket -> TB002-500-02BE
- J2, J3: value Conn_01x02_Socket -> JST_XH_S2B-XH-A-1
- Q1: value Q_PMOS_DSG -> BSS84PH6327XTSA2
- R10, R7: value 510R -> 910R
- R5: value 1.8kR -> 4.3kR
- R8: value 560R -> 510R
- SW1, SW2: value SW_SPDT -> OS102011MS2QN1
- moved R2 3.66 mm to (96.5, 72.4)
- moved R9 3.00 mm to (96.2, 77.0)
- moved Q1 2.91 mm to (100.1, 76.1), turned to 0 degrees
- moved C14 2.65 mm to (96.2, 75.4)
- moved U2 2.10 mm to (100.2, 72.4), turned to 180 degrees
- moved R15 0.83 mm to (78.3, 77.0)
- moved C9 0.38 mm to (139.8, 60.2)
- moved J3 0.30 mm to (176.4, 79.8)
- moved C6 0.28 mm to (139.8, 63.5)
- moved J2 0.20 mm to (176.3, 63.8)
- moved C5 0.12 mm to (141.6, 63.7)
Connections:
- Q1 pad 1: /Phone Charging/CHG_EN -> /Phone Charging/CURR_LIM_nFLT
- Q1 pad 3: /Phone Charging/CURR_LIM_nFLT -> /Phone Charging/CHG_EN
- U2 pad 1: VLIM_5V -> VSYS_5V
- U2 pad 2: Net-(U2-ILIM) -> GND
- U2 pad 5: GND -> Net-(U2-ILIM)
- U2 pad 6: VSYS_5V -> VLIM_5V
Routing:
- net /12V to 5V/12V_SW: track 0.00 -> 5.57 mm
- net /Phone Charging/CURR_LIM_nFLT: track 5.21 -> 10.7 mm
- net /Phone Charging/CHG_EN: track 29.3 -> 34.7 mm
- net VLIM_5V: track 14.5 -> 19.1 mm
- net Net-(C7-Pad1): track 0.00 -> 3.48 mm
- net Net-(J4-CC2): track 0.00 -> 3.03 mm
- net Net-(Q1-S): track 9.08 -> 10.2 mm
- net GND: track 4.65 -> 5.62 mm, vias 5 -> 126
- net Net-(U2-ILIM): track 2.64 -> 2.03 mm
Other:
- board text added: "Power V1 Designed by Olivia Ye 02/21/2026"
- board text added: "roamr"
