File: hw/roamr-power/phone_charging.kicad_sch (KiCad schematic)
At the start: 12 parts, among them Q1 Q_PMOS_DSG, SW1 SW_SPDT, U2 TPS2553DDBVR

Commit message: final edits
Parts:
- removed Q1: Q_PMOS_DSG, BSS84PH6327XTSA2:SOT95P240X110-3N, symbol Transistor_FET:Q_PMOS_DSG
- added Q1: BSS84PH6327XTSA2, BSS84PH6327XTSA2:SOT95P240X110-3N, symbol BSS84PH6327XTSA2:BSS84PH6327XTSA2
- D2: footprint KT_EELP41.12-S2U1-25-2X4X-5-R18:KTEELP4112S2U1252X4X5R18 -> KT-0603:LEDC1608X70N; Manufacturer_Part_Number (none) -> KT-0603G
- D3: footprint KR_DELPS1.22-VGVI-23-H3Q4:KRDELPS122VGVI23H3Q4 -> KT-0603:LEDC1608X70N; Manufacturer_Part_Number (none) -> KT-0603R
- R7: value 510R -> 910R
- R8: value 560R -> 510R
- SW1: value SW_SPDT -> OS102011MS2QN1; Manufacturer_Part_Number (none) -> OS102011MS2QN1
- U2: Manufacturer_Part_Number (none) -> TPS2553DDBVR
Connections:
- net CHG_EN: now also Q1.3 (D)
- net CURR_LIM_nFLT: now also Q1.1 (G)
- net GND: now also U2.2 (GND); no longer U2.5 (GND), U2.7 (EPAD)
- net VLIM_5V: now also U2.6 (OUT); no longer U2.1 (OUT)
- net VSYS_5V: now also U2.1 (IN); no longer U2.6 (IN)
- net at R2.1: now also U2.5 (ILIM); no longer U2.2 (ILIM)
- net at R8.1: now also Q1.2 (S)
Other:
- note added: "2.4Vf"
- note added: "3.1Vf"
- note removed: "2.5Vf"
Changed lines of the file:
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@@
 		)
 	)
-	(text "2.5Vf"
+	(text "3.1Vf\n"
 		(exclude_from_sim no)
 		(at 107.95 149.86 0)
@@
 		)
 	)
+	(text "2.4Vf\n"
+		(exclude_from_sim no)
+		(at 181.61 152.4 0)
+		(effects
+			(font
+				(size 1.27 1.27)
+			)
+		)
+	)
 	(text "Fault Indicator"
 		(exclude_from_sim no)
@@
 	)
 	(junction
-		(at 158.75 67.31)
-		(diameter 0)
-		(color 0 0 0 0)
-	)
-	(junction
 		(at 115.57 64.77)
 		(diameter 0)
@@
 	(wire
 		(pts
-			(xy 165.1 120.65) (xy 175.26 120.65)
+			(xy 165.1 116.84) (xy 175.26 116.84)
 		)
 		(stroke
@@
 	(wire
 		(pts
-			(xy 158.75 67.31) (xy 158.75 74.93)
+			(xy 158.75 64.77) (xy 158.75 74.93)
 		)
 		(stroke
@@
 	(wire
 		(pts
-			(xy 158.75 64.77) (xy 158.75 67.31)
-		)
-		(stroke
-			(width 0)
-			(type default)
-		)
-	)
-	(wire
-		(pts
 			(xy 105.41 58.42) (xy 115.57 58.42)
 		)
@@
 	(wire
 		(pts
-			(xy 175.26 120.65) (xy 175.26 124.46)
+			(xy 175.26 116.84) (xy 175.26 119.38)
 		)
 		(stroke
@@
 		(pts
 			(xy 81.28 124.46) (xy 86.36 124.46)
-		)
-		(stroke
-			(width 0)
-			(type default)
-		)
-	)
-	(wire
-		(pts
-			(xy 158.75 67.31) (xy 156.21 67.31)
 		)
 		(stroke
@@
 	)
 	(label "CHG_EN"
-		(at 165.1 120.65 180)
+		(at 165.1 116.84 180)
 		(effects
 			(font
@@
 			)
 		)
-		(pin "7"
+		(property "Manufacturer_Part_Number" "TPS2553DDBVR"
+			(at 114.3 57.15 0)
+			(effects
+				(font
+					(size 1.27 1.27)
+				)
+				(hide yes)
+			)
 		)
 		(pin "3"
@@
 			)
 		)
-		(property "Footprint" "KT_EELP41.12-S2U1-25-2X4X-5-R18:KTEELP4112S2U1252X4X5R18"
+		(property "Footprint" "KT-0603:LEDC1608X70N"
 			(at 101.6 143.51 0)
 			(effects
@@
 			)
 		)
+		(property "Manufacturer_Part_Number" "KT-0603G"
+			(at 101.6 143.51 90)
+			(effects
+				(font
+					(size 1.27 1.27)
+				)
+				(hide yes)
+			)
+		)
 		(pin "1"
 		)
@@
 				(path "/bfe84b16-3df2-48dd-882e-523c3a68f778/7cadbd84-e43d-43ba-a052-9e62bf6faf2f"
 					(reference "#PWR016")
-					(unit 1)
-				)
-			)
-		)
-	)
-	(symbol
-		(lib_id "Transistor_FET:Q_PMOS_DSG")
-		(at 172.72 129.54 0)
-		(unit 1)
-		(exclude_from_sim no)
-		(in_bom yes)
-		(on_board yes)
-		(dnp no)
-		(property "Reference" "Q1"
-			(at 179.07 129.54 0)
-			(effects
-				(font
-					(size 1.27 1.27)
-				)
-				(justify left)
-			)
-		)
-		(property "Value" "Q_PMOS_DSG"
-			(at 179.07 130.8099 0)
-			(effects
-				(font
-					(size 1.27 1.27)
-				)
-				(justify left)
-				(hide yes)
-			)
-		)
-		(property "Footprint" "BSS84PH6327XTSA2:SOT95P240X110-3N"
-			(at 177.8 127 0)
-			(effects
-				(font
-					(size 1.27 1.27)
-				)
-				(hide yes)
-			)
-		)
-		(property "Datasheet" "~"
-			(at 172.72 129.54 0)
-			(effects
-				(font
-					(size 1.27 1.27)
-				)
-				(hide yes)
-			)
-		)
-		(property "Description" "P-MOSFET transistor, drain/source/gate"
-			(at 172.72 129.54 0)
-			(effects
-				(font
-					(size 1.27 1.27)
-				)
-				(hide yes)
-			)
-		)
-		(pin "2"
-		)
-		(pin "3"
-		)
-		(pin "1"
-		)
-		(instances
-			(project ""
-				(path "/bfe84b16-3df2-48dd-882e-523c3a68f778/7cadbd84-e43d-43ba-a052-9e62bf6faf2f"
-					(reference "Q1")
 					(unit 1)
 				)
@@
 			)
 		)
-		(property "Footprint" "KR_DELPS1.22-VGVI-23-H3Q4:KRDELPS122VGVI23H3Q4"
+		(property "Footprint" "KT-0603:LEDC1608X70N"
 			(at 175.26 146.05 0)
 			(effects
@@
 		(property "Sim.Pins" "1=K 2=A"
 			(at 175.26 146.05 0)
+			(effects
+				(font
+					(size 1.27 1.27)
+				)
+				(hide yes)
+			)
+		)
+		(property "Manufacturer_Part_Number" "KT-0603R"
+			(at 175.26 146.05 90)
 			(effects
 				(font
@@
 			)
 		)
-		(property "Value" "560R"
+		(property "Value" "510R"
 			(at 177.8 139.6999 0)
 			(effects
@@
 		(on_board yes)
 		(dnp no)
-		(fields_autoplaced yes)
 		(property "Reference" "SW1"
 			(at 91.44 115.57 0)
@@
 			)
 		)
-		(property "Value" "SW_SPDT"
-			(at 91.44 118.11 0)
+		(property "Value" "OS102011MS2QN1"
+			(at 96.52 118.11 0)
 			(effects
 				(font
@@
 			)
 		)
+		(property "Manufacturer_Part_Number" "OS102011MS2QN1"
+			(at 91.44 124.46 0)
+			(effects
+				(font
+					(size 1.27 1.27)
+				)
+				(hide yes)
+			)
+		)
 		(pin "2"
 		)
@@
 				(path "/bfe84b16-3df2-48dd-882e-523c3a68f778/7cadbd84-e43d-43ba-a052-9e62bf6faf2f"
 					(reference "SW1")
+					(unit 1)
+				)
+			)
+		)
+	)
+	(symbol
+		(lib_id "BSS84PH6327XTSA2:BSS84PH6327XTSA2")
+		(at 167.64 129.54 0)
+		(unit 1)
+		(exclude_from_sim no)
+		(in_bom yes)
+		(on_board yes)
+		(dnp no)
+		(fields_autoplaced yes)
+		(property "Reference" "Q1"
+			(at 179.07 125.7299 0)
+			(effects
+				(font
+					(size 1.27 1.27)
+				)
+				(justify left)
+			)
+		)
+		(property "Value" "BSS84PH6327XTSA2"
+			(at 179.07 128.2699 0)
+			(effects
+				(font
+					(size 1.27 1.27)
+				)
+				(justify left)
+			)
+		)
+		(property "Footprint" "BSS84PH6327XTSA2:SOT95P240X110-3N"
+			(at 179.07 228.27 0)
+			(effects
+				(font
+					(size 1.27 1.27)
+				)
+				(justify left top)
+				(hide yes)
+			)
+		)
+		(property "Datasheet" "https://componentsearchengine.com/Datasheets/2/BSS84PH6327XTSA2.pdf"
+			(at 179.07 328.27 0)
+			(effects
+				(font
+					(size 1.27 1.27)
+				)
+				(justify left top)
+				(hide yes)
+			)
+		)
+		(property "Description" "INFINEON - BSS84PH6327XTSA2 - MOSFET, P, -60V, -0.17A, SOT-23"
+			(at 167.64 129.54 0)
+			(effects
+				(font
+					(size 1.27 1.27)
+				)
+				(hide yes)
+			)
+		)
+		(property "Height" "1.1"
+			(at 179.07 528.27 0)
+			(effects
+				(font
+					(size 1.27 1.27)
+				)
+				(justify left top)
+				(hide yes)
+			)
+		)
+		(property "Mouser Part Number" "726-BSS84PH6327XTSA2"
+			(at 179.07 628.27 0)
+			(effects
+				(font
+					(size 1.27 1.27)
+				)
+				(justify left top)
+				(hide yes)
+			)
+		)
+		(property "Mouser Price/Stock" "https://www.mouser.co.uk/ProductDetail/Infineon-Technologies/BSS84PH6327XTSA2?qs=K00xGehIljvU09gSF2VpyQ%3D%3D"
+			(at 179.07 728.27 0)
+			(effects
+				(font
+					(size 1.27 1.27)
+				)
+				(justify left top)
+				(hide yes)
+			)
+		)
+		(property "Manufacturer_Name" "Infineon"
+			(at 179.07 828.27 0)
+			(effects
+				(font
+					(size 1.27 1.27)
+				)
+				(justify left top)
+				(hide yes)
+			)
+		)
+		(property "Manufacturer_Part_Number" "BSS84PH6327XTSA2"
+			(at 179.07 928.27 0)
+			(effects
+				(font
+					(size 1.27 1.27)
+				)
+				(justify left top)
+				(hide yes)
+			)
+		)
+		(pin "3"
+		)
+		(pin "1"
+		)
+		(pin "2"
+		)
+		(instances
+			(project ""
+				(path "/bfe84b16-3df2-48dd-882e-523c3a68f778/7cadbd84-e43d-43ba-a052-9e62bf6faf2f"
+					(reference "Q1")
 					(unit 1)
 				)
@@
 			)
 		)
-		(property "Value" "510R"
+		(property "Value" "910R"
 			(at 104.14 134.6199 0)
 			(effects
