File: hw/roamr-motors/bldc_driver.kicad_sch (KiCad schematic)
At the start: 14 parts, among them U4 DRV8316CRRGFR

Commit message: final
Parts:
- C15: value 47uF -> 47nF
Changed lines of the file:
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@@
 			)
 		)
-		(property "Value" "47uF"
+		(property "Value" "47nF"
 			(at 57.15 48.26 90)
 			(effects
