File: hw/roamr-motors/roamr-motors.kicad_sch (KiCad schematic)
At the start: 26 parts, among them J1 JST_XH_S2B-XH-A-1, J10 JST_SH_BM06B-SRSS-TB, J2 USB4215-03-A, J3 USB4215-03-A, J4 JST_XH_S2B-XH-A-1, J5 JST_XH_S2B-XH-A-1, J6 JST_PH_B3B-PH-SM4-TB, J7 JST_SH_BM06B-SRSS-TB, J8 JST_XH_S2B-XH-A-1, J9 JST_PH_B3B-PH-SM4-TB

Commit message: outputs and last minute updates
Parts:
- D1, D4: value SMLJ12A-R -> SMLJ13CA-R; footprint SMLJ12A-R:DIOM7959X262N -> SMLJ13CA-R:DIOM7959X262N; Manufacturer_Part_Number (none) -> SMLJ13CA-R
- D2, D3, D5, D6, D7, D8: Manufacturer_Part_Number (none) -> LESD5D5.0CT1G
- F1, F2: Manufacturer_Part_Number (none) -> 0466005.NRHF
- J1, J4, J5, J8: Manufacturer_Part_Number (none) -> JST_XH_S2B-XH-A-1
- J10, J7: Manufacturer_Part_Number (none) -> JST_SH_BM06B-SRSS-TB
- J2, J3: Manufacturer_Part_Number (none) -> USB4215-03-A
- J6, J9: Manufacturer_Part_Number (none) -> JST_PH_B3B-PH-SM4-TB
