File: hw/roamr-motors/roamr-motors.kicad_pcb (KiCad board)
At the start: 4 copper layers, 115 x 55 mm, 110 parts, among them J1 JST_XH_S2B-XH-A-1, J10 JST_SH_BM06B-SRSS-TB, J2 USB4215-03-A, J3 USB4215-03-A, J4 JST_XH_S2B-XH-A-1, J5 JST_XH_S2B-XH-A-1, J6 JST_PH_B3B-PH-SM4-TB, J7 JST_SH_BM06B-SRSS-TB, J8 JST_XH_S2B-XH-A-1, J9 JST_PH_B3B-PH-SM4-TB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

Commit message: final
Parts:
- C15, C24: value 47uF -> 47nF
